File: PCB/Original/ultraHex-master/ultraHex-master/_restore_backup_2026-07-17T15-32-36-407/bm1366-1.kicad_sch (KiCad schematic)
At the start: 55 parts, among them U10 SGM2036-0v8, U11 SGM2036-1v8, U12 BM1366_mode1, U13 BM1366_mode1, U14 25MHz

Commit message: PCBLayout完成
Parts:
- renumbered C63 to C10, C65 to C11, C56 to C12, C72 to C12, C68 to C13, C55 to C14, C74 to C14, C57 to C15, C75 to C15, C76 to C16, C58 to C16, C77 to C17, C59 to C17, C61 to C18, C78 to C18, C45 to C2, C64 to C2, C53 to C24, C54 to C24, C46 to C3, C66 to C3, C67 to C4, C47 to C4, C48 to C5, C70 to C5, C69 to C6, C49 to C6, C71 to C8, C62 to C8, C52 to C8, C73 to C8, C51 to C8, C60 to C8, C50 to C8, R33 to R6, R28 to R6, TP35 to TP13, TP37 to TP13, TP34 to TP13, TP33 to TP13, TP39 to TP13, TP40 to TP13, TP38 to TP13, TP41 to TP13, TP36 to TP13, U14 to U1, U12 to U14, U13 to U14
