File: PCB/Original/ultraHex-master/ultraHex-master/_restore_backup_2026-07-17T15-32-36-407/bm1366-2.kicad_sch (KiCad schematic)
At the start: 74 parts, among them U15 TLV3544, U16 SGM2036-1v8, U17 SGM2036-0v8, U18 BM1366_mode0, U19 25MHz, U20 BM1366_mode0

Commit message: PCBLayout完成
Parts:
- renumbered C97 to C10, C99 to C11, C90 to C12, C107 to C12, C101 to C13, C89 to C14, C110 to C14, C92 to C14, C91 to C15, C108 to C15, C113 to C16, C109 to C17, C94 to C17, C96 to C18, C114 to C18, C98 to C2, C79 to C2, C88 to C24, C87 to C24, C100 to C3, C80 to C3, C102 to C4, C81 to C4, C83 to C5, C104 to C5, C103 to C6, C85 to C6, C84 to C8, C95 to C8, C86 to C8, C111 to C8, C112 to C8, C106 to C8, C82 to C8, C105 to C8, C93 to C8, R46 to R6, R52 to R6, R43 to R6, R35 to R6, R37 to R6, R49 to R6, R47 to R6, R54 to R6, R42 to R6, R51 to R6, R36 to R6, R34 to R6, R53 to R6, R48 to R6, R45 to R6, R55 to R6, R44 to R6, R50 to R6, TP43 to TP13, TP50 to TP13, TP42 to TP13, TP45 to TP13, TP48 to TP13, TP49 to TP13, TP46 to TP13, TP44 to TP13, TP47 to TP13, U19 to U1
