File: PCB/Original/ultraHex-master/ultraHex-master/_restore_backup_2026-07-17T15-32-36-407/bm1366-3.kicad_sch (KiCad schematic)
At the start: 79 parts, among them U21 TLV3544, U22 BM1366_mode1, U23 SGM2036-0v8, U24 SGM2036-1v8, U25 BM1366_mode1, U26 25MHz

Commit message: PCBLayout完成
Parts:
- renumbered C134 to C10, C137 to C11, C143 to C12, C124 to C12, C140 to C13, C123 to C14, C146 to C14, C127 to C15, C144 to C15, C128 to C16, C149 to C16, C145 to C17, C129 to C17, C150 to C18, C131 to C18, C133 to C2, C115 to C2, C126 to C24, C125 to C24, C135 to C3, C116 to C3, C136 to C4, C117 to C4, C139 to C5, C118 to C5, C138 to C6, C119 to C6, C120 to C8, C132 to C8, C148 to C8, C130 to C8, C147 to C8, C142 to C8, C141 to C8, C122 to C8, C121 to C8, R73 to R6, R61 to R6, R72 to R6, R76 to R6, R71 to R6, R68 to R6, R69 to R6, R56 to R6, R75 to R6, R70 to R6, R58 to R6, R57 to R6, R62 to R6, R59 to R6, R67 to R6, R74 to R6, R60 to R6, R77 to R6, TP63 to TP13, TP60 to TP13, TP59 to TP13, TP58 to TP13, TP61 to TP13, TP56 to TP13, TP54 to TP13, TP62 to TP13, TP52 to TP13, TP51 to TP13, TP53 to TP13, TP55 to TP13, TP57 to TP13, U26 to U1, U25 to U14, U22 to U14
