File: PCB/Original/ultraHex-master/ultraHex-master/_restore_backup_2026-07-17T15-32-36-407/esp32.kicad_sch (KiCad schematic)
At the start: 53 parts, among them J4 TC2030-IDC, J5 Conn_01x04, J6 Conn_01x06, J7 USB_C_Receptacle_USB2.0, SW1 SWITCH-SPST, SW2 SWITCH-SPST, U5 SN74AVC4T774, U6 ESP32-S3-WROOM-1, Y1 32.768kHz

Commit message: PCBLayout完成
Parts:
- renumbered C35 to C25, C34 to C25, C32 to C50, J7 to J8, R18 to R20, R22 to R3, R23 to R5, R21 to R8
