File: PCB/Original/ultraHex-master/ultraHex-master/_restore_backup_2026-07-17T15-32-36-407/fan.kicad_sch (KiCad schematic)
At the start: 16 parts, among them J8 Conn_01x04, J9 Conn_01x04, U7 TMP1075, U8 TMP1075, U9 EMC2302

Commit message: PCBLayout完成
Parts:
- renumbered R27 to R7, R26 to R7
