File: PCB/Original/ultraHex-master/ultraHex-master/_restore_backup_2026-07-17T15-32-36-407/power.kicad_sch (KiCad schematic)
At the start: 65 parts, among them J3 Conn_02x05_Odd_Even, T1 net-tie, U1 LMR54410, U2 RT9080-33GJ5, U3 TPS546D24ARVFR, U4 MIC5504

Commit message: PCBLayout完成
Parts:
- renumbered C12 to C8, C6 to C8, R3 to R6, R1 to R6, R2 to R6, R17 to R7
